File: AGV.brd (EAGLE design)
At the start: 80.7 x 76.3 mm, 10 parts

Commit message: reubicación de orificios para tornillos
Changed lines of the file:
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@@
 <layer number="27" name="tValues" color="7" fill="1" visible="yes" active="yes"/>
 <layer number="28" name="bValues" color="7" fill="1" visible="yes" active="yes"/>
-<layer number="29" name="tStop" color="7" fill="3" visible="no" active="yes"/>
-<layer number="30" name="bStop" color="7" fill="6" visible="no" active="yes"/>
-<layer number="31" name="tCream" color="7" fill="4" visible="no" active="yes"/>
-<layer number="32" name="bCream" color="7" fill="5" visible="no" active="yes"/>
-<layer number="33" name="tFinish" color="6" fill="3" visible="no" active="yes"/>
-<layer number="34" name="bFinish" color="6" fill="6" visible="no" active="yes"/>
-<layer number="35" name="tGlue" color="7" fill="4" visible="no" active="yes"/>
-<layer number="36" name="bGlue" color="7" fill="5" visible="no" active="yes"/>
-<layer number="37" name="tTest" color="7" fill="1" visible="no" active="yes"/>
-<layer number="38" name="bTest" color="7" fill="1" visible="no" active="yes"/>
+<layer number="29" name="tStop" color="7" fill="3" visible="yes" active="yes"/>
+<layer number="30" name="bStop" color="7" fill="6" visible="yes" active="yes"/>
+<layer number="31" name="tCream" color="7" fill="4" visible="yes" active="yes"/>
+<layer number="32" name="bCream" color="7" fill="5" visible="yes" active="yes"/>
+<layer number="33" name="tFinish" color="6" fill="3" visible="yes" active="yes"/>
+<layer number="34" name="bFinish" color="6" fill="6" visible="yes" active="yes"/>
+<layer number="35" name="tGlue" color="7" fill="4" visible="yes" active="yes"/>
+<layer number="36" name="bGlue" color="7" fill="5" visible="yes" active="yes"/>
+<layer number="37" name="tTest" color="7" fill="1" visible="yes" active="yes"/>
+<layer number="38" name="bTest" color="7" fill="1" visible="yes" active="yes"/>
 <layer number="39" name="tKeepout" color="4" fill="11" visible="yes" active="yes"/>
 <layer number="40" name="bKeepout" color="1" fill="11" visible="yes" active="yes"/>
@@
 <layer number="42" name="bRestrict" color="1" fill="10" visible="yes" active="yes"/>
 <layer number="43" name="vRestrict" color="2" fill="10" visible="yes" active="yes"/>
-<layer number="44" name="Drills" color="7" fill="1" visible="no" active="yes"/>
+<layer number="44" name="Drills" color="7" fill="1" visible="yes" active="yes"/>
 <layer number="45" name="Holes" color="7" fill="1" visible="yes" active="yes"/>
-<layer number="46" name="Milling" color="3" fill="1" visible="no" active="yes"/>
+<layer number="46" name="Milling" color="3" fill="1" visible="yes" active="yes"/>
 <layer number="47" name="Measures" color="7" fill="1" visible="yes" active="yes"/>
 <layer number="48" name="Document" color="7" fill="1" visible="yes" active="yes"/>
@@
 <wire x1="0.11948125" y1="76.2708" x2="0.02184375" y2="0.020575" width="0" layer="20"/>
 <hole x="19.892771875" y="3.393159375" drill="1"/>
-<hole x="19.892771875" y="3.393159375" drill="1"/>
+<hole x="19.892771875" y="3.393159375" drill="3.048"/>
 <hole x="61.81206875" y="3.437053125" drill="1"/>
-<hole x="61.81206875" y="3.437053125" drill="1"/>
-<hole x="20.12835625" y="23.471071875" drill="1"/>
-<hole x="70.345071875" y="39.53631875" drill="1"/>
+<hole x="61.81206875" y="3.437053125" drill="3.048"/>
+<hole x="23.050703125" y="23.74293125" drill="3.048"/>
+<hole x="72.763915625" y="39.819475" drill="3.048"/>
+<hole x="19.949771875" y="71.639178125" drill="3.048"/>
 </plain>
 <attributes>
@@
 <wire x1="48.6726" y1="70.128465625" x2="37.93225625" y2="70.09608125" width="0" layer="19" extent="1-1"/>
 <wire x1="66.67136875" y1="46.04328125" x2="48.89136875" y2="46.04328125" width="0" layer="19" extent="1-1"/>
+<wire x1="66.67136875" y1="18.10328125" x2="66.67136875" y2="46.04328125" width="0" layer="19" extent="1-1"/>
 </signal>
 <signal name="+3V3">
